File: circuit/power_supply/power-supply.sch (KiCad schematic (older format))
At the start: 16 parts

Commit message: power_supply: filled the value in all components
Parts:
- 2SK2611: renamed from Q?; value MOS_N -> MOSFET-N
- C1: renamed from C?; value CP1 -> 100uf/16v
- C2: renamed from C?; value C -> 1500pf
- C3: renamed from C?; value CP1 -> 33v/250v
- C4: renamed from C?; value CP1 -> 33uf/250v
- D1: renamed from D?; value DIODE -> 1N4148
- D2: renamed from D?; value DIODE -> FR157
- L1: renamed from L?; value INDUCTOR -> 220uh
- L2: renamed from L?; value INDUCTOR -> 22uh
- R1, R2: renamed from R?; value R -> 1k ohm
- R3: renamed from R?; value R -> 620 ohm
- R4: renamed from R?; value R -> 100k ohm
- R5: renamed from R?; value R -> 760 ohm
- gave numbers to parts that had none: 2
Connections:
- net labels added: +12V
- net labels removed: 12V
Changed lines of the file:
@@
-EESchema Schematic File Version 2  date 2014年02月01日 (週六) 20時24分48秒
+EESchema Schematic File Version 2  date 2014年02月01日 (週六) 21時19分31秒
 LIBS:power
 LIBS:device
@@
 LIBS:valves
 LIBS:power-custom
-LIBS:power-supply-cache
 EELAYER 25  0
 EELAYER END
@@
 encoding utf-8
 Sheet 1 1
-Title ""
+Title "Nixie tube power supply"
 Date "1 feb 2014"
 Rev ""
-Comp ""
+Comp "Sigma Lab"
 Comment1 ""
 Comment2 ""
@@
 	3350 4750 3350 5000
 Text GLabel 2600 3100 0    60   Input ~ 0
-12V
-$Comp
-L INDUCTOR L?
++12V
+$Comp
+L INDUCTOR L2
 U 1 1 52ECE279
 P 8400 3100
-F 0 "L?" V 8350 3100 40  0000 C CNN
-F 1 "INDUCTOR" V 8500 3100 40  0000 C CNN
+F 0 "L2" V 8350 3100 40  0000 C CNN
+F 1 "22uh" V 8500 3100 40  0000 C CNN
 	1    8400 3100
 	0    -1   -1   0
 $EndComp
 $Comp
-L INDUCTOR L?
+L INDUCTOR L1
 U 1 1 52ECE276
 P 6250 3100
-F 0 "L?" V 6200 3100 40  0000 C CNN
-F 1 "INDUCTOR" V 6350 3100 40  0000 C CNN
+F 0 "L1" V 6200 3100 40  0000 C CNN
+F 1 "220uh" V 6350 3100 40  0000 C CNN
 	1    6250 3100
 	0    -1   -1   0
@@
 +170V
 $Comp
-L GND #PWR01
+L GND #PWR2
 U 1 1 52ECE132
 P 9200 5000
-F 0 "#PWR01" H 9200 5000 30  0001 C CNN
+F 0 "#PWR2" H 9200 5000 30  0001 C CNN
 F 1 "GND" H 9200 4930 30  0001 C CNN
 	1    9200 5000
@@
 $EndComp
 $Comp
-L R R?
+L R R5
 U 1 1 52ECE108
 P 7650 4500
-F 0 "R?" V 7730 4500 50  0000 C CNN
-F 1 "R" V 7650 4500 50  0000 C CNN
+F 0 "R5" V 7730 4500 50  0000 C CNN
+F 1 "760 ohm" V 7650 4500 50  0000 C CNN
 	1    7650 4500
 	1    0    0    -1
 $EndComp
 $Comp
-L R R?
+L R R4
 U 1 1 52ECE106
 P 7650 3700
-F 0 "R?" V 7730 3700 50  0000 C CNN
-F 1 "R" V 7650 3700 50  0000 C CNN
+F 0 "R4" V 7730 3700 50  0000 C CNN
+F 1 "100k ohm" V 7650 3700 50  0000 C CNN
 	1    7650 3700
 	1    0    0    -1
 $EndComp
 $Comp
-L R R?
+L R R3
 U 1 1 52ECE103
 P 5200 3350
-F 0 "R?" V 5280 3350 50  0000 C CNN
-F 1 "R" V 5200 3350 50  0000 C CNN
+F 0 "R3" V 5280 3350 50  0000 C CNN
+F 1 "620 ohm" V 5200 3350 50  0000 C CNN
 	1    5200 3350
 	1    0    0    -1
 $EndComp
 $Comp
-L R R?
+L R R1
 U 1 1 52ECE101
 P 4050 3350
-F 0 "R?" V 4130 3350 50  0000 C CNN
-F 1 "R" V 4050 3350 50  0000 C CNN
+F 0 "R1" V 4130 3350 50  0000 C CNN
+F 1 "1k ohm" V 4050 3350 50  0000 C CNN
 	1    4050 3350
 	1    0    0    -1
 $EndComp
 $Comp
-L R R?
+L R R2
 U 1 1 52ECE0FB
 P 4200 4750
-F 0 "R?" V 4280 4750 50  0000 C CNN
-F 1 "R" V 4200 4750 50  0000 C CNN
+F 0 "R2" V 4280 4750 50  0000 C CNN
+F 1 "1k ohm" V 4200 4750 50  0000 C CNN
 	1    4200 4750
 	1    0    0    -1
 $EndComp
 $Comp
-L CP1 C?
+L CP1 C4
 U 1 1 52ECE0DF
 P 8700 4050
-F 0 "C?" H 8750 4150 50  0000 L CNN
-F 1 "CP1" H 8750 3950 50  0000 L CNN
+F 0 "C4" H 8750 4150 50  0000 L CNN
+F 1 "33uf/250v" H 8750 3950 50  0000 L CNN
 	1    8700 4050
 	1    0    0    -1
 $EndComp
 $Comp
-L CP1 C?
+L CP1 C3
 U 1 1 52ECE0D9
 P 8100 4050
-F 0 "C?" H 8150 4150 50  0000 L CNN
-F 1 "CP1" H 8150 3950 50  0000 L CNN
+F 0 "C3" H 8150 4150 50  0000 L CNN
+F 1 "33v/250v" H 8150 3950 50  0000 L CNN
 	1    8100 4050
 	1    0    0    -1
 $EndComp
 $Comp
-L DIODE D?
+L DIODE D1
 U 1 1 52ECE0D3
 P 6050 3600
-F 0 "D?" H 6050 3700 40  0000 C CNN
-F 1 "DIODE" H 6050 3500 40  0000 C CNN
+F 0 "D1" H 6050 3700 40  0000 C CNN
+F 1 "1N4148" H 6050 3500 40  0000 C CNN
 	1    6050 3600
 	1    0    0    -1
 $EndComp
 $Comp
-L DIODE D?
+L DIODE D2
 U 1 1 52ECE0D1
 P 7300 3100
-F 0 "D?" H 7300 3200 40  0000 C CNN
-F 1 "DIODE" H 7300 3000 40  0000 C CNN
+F 0 "D2" H 7300 3200 40  0000 C CNN
+F 1 "FR157" H 7300 3000 40  0000 C CNN
 	1    7300 3100
 	1    0    0    -1
 $EndComp
 $Comp
-L PNP Q?
+L PNP 2SB647
 U 1 1 52ECE0A1
 P 6300 4100
-F 0 "Q?" H 6300 3950 60  0000 R CNN
-F 1 "PNP" H 6300 4250 60  0000 R CNN
+F 0 "2SB647" H 6300 4400 60  0000 R CNN
+F 1 "PNP" H 6200 4300 60  0000 R CNN
 	1    6300 4100
 	1    0    0    1
 $EndComp
 $Comp
-L C C?
+L C C2
 U 1 1 52ECE02C
 P 3350 4550
-F 0 "C?" H 3400 4650 50  0000 L CNN
-F 1 "C" H 3400 4450 50  0000 L CNN
+F 0 "C2" H 3400 4650 50  0000 L CNN
+F 1 "1500pf" H 3400 4450 50  0000 L CNN
 	1    3350 4550
 	1    0    0    -1
 $EndComp
 $Comp
-L CP1 C?
+L CP1 C1
 U 1 1 52ECE01C
 P 2850 4200
-F 0 "C?" H 2900 4300 50  0000 L CNN
-F 1 "CP1" H 2900 4100 50  0000 L CNN
+F 0 "C1" H 2900 4300 50  0000 L CNN
+F 1 "100uf/16v" H 2900 4100 50  0000 L CNN
 	1    2850 4200
 	1    0    0    -1
 $EndComp
 $Comp
-L MOS_N Q?
+L MOS_N 2SK2611
 U 1 1 52ECDF19
 P 6850 3600
-F 0 "Q?" H 6860 3770 60  0000 R CNN
-F 1 "MOS_N" H 6860 3450 60  0000 R CNN
+F 0 "2SK2611" H 6750 3750 60  0000 R CNN
+F 1 "MOSFET-N" H 6800 3850 60  0000 R CNN
 	1    6850 3600
 	1    0    0    -1
 $EndComp
 $Comp
-L MCS34063A U?
+L MCS34063A U1
 U 1 1 52ECDE52
 P 4600 4050
-F 0 "U?" H 4300 4600 60  0000 C CNN
+F 0 "U1" H 4300 4600 60  0000 C CNN
 F 1 "MCS34063A" H 4700 4600 60  0000 C CNN
 	1    4600 4050
@@
 $EndComp
 $Comp
-L GND #PWR02
+L GND #PWR1
 U 1 1 52ECDB44
 P 2450 5000
-F 0 "#PWR02" H 2450 5000 30  0001 C CNN
+F 0 "#PWR1" H 2450 5000 30  0001 C CNN
 F 1 "GND" H 2450 4930 30  0001 C CNN
 	1    2450 5000

Commit message: power_supply: replaced the components of Vcc/Ground
Connections:
- net labels added: GNDPWR
- net labels removed: GND
- wire segments 41 -> 59
Changed lines of the file:
@@
-EESchema Schematic File Version 2  date 2014年02月01日 (週六) 21時19分31秒
+EESchema Schematic File Version 2  date 2014年02月01日 (週六) 21時51分08秒
 LIBS:power
 LIBS:device
@@
 LIBS:valves
 LIBS:power-custom
+LIBS:power-supply-cache
 EELAYER 25  0
 EELAYER END
@@
 Comment4 ""
 $EndDescr
-Wire Wire Line
-	9200 5000 2450 5000
+$Comp
+L GNDPWR #PWR?
+U 1 1 52ECFBB9
+P 2600 5000
+F 0 "#PWR?" H 2600 5050 40  0001 C CNN
+F 1 "GNDPWR" H 2600 4920 40  0000 C CNN
+	1    2600 5000
+	0    1    1    0
+$EndComp
+$Comp
+L +12V #PWR?
+U 1 1 52ECFBAD
+P 2600 3100
+F 0 "#PWR?" H 2600 3050 20  0001 C CNN
+F 1 "+12V" H 2600 3200 30  0000 C CNN
+	1    2600 3100
+	0    -1   -1   0
+$EndComp
+Wire Wire Line
+	8700 5000 8100 5000
+Wire Wire Line
+	8100 5000 7650 5000
+Wire Wire Line
+	7650 5000 6950 5000
+Wire Wire Line
+	6950 5000 6400 5000
+Wire Wire Line
+	6400 5000 4200 5000
+Wire Wire Line
+	4200 5000 3800 5000
+Wire Wire Line
+	3800 5000 3350 5000
+Wire Wire Line
+	3350 5000 2850 5000
+Wire Wire Line
+	2850 5000 2600 5000
 Wire Wire Line
 	3350 4350 3350 4000
@@
 	2850 2900 5600 2900
 Wire Wire Line
-	2850 2900 2850 4000
+	2850 2900 2850 3100
+Wire Wire Line
+	2850 3100 2850 4000
 Connection ~ 2850 5000
 Wire Wire Line
@@
 	8100 3850 8100 3100
 Wire Wire Line
-	7100 3100 6550 3100
-Wire Wire Line
-	8100 3100 7500 3100
+	7100 3100 6950 3100
+Wire Wire Line
+	6950 3100 6550 3100
+Wire Wire Line
+	8100 3100 7650 3100
+Wire Wire Line
+	7650 3100 7500 3100
 Wire Wire Line
 	8700 3100 8700 3850
 Wire Wire Line
-	7650 4250 7650 3950
-Wire Wire Line
-	6250 3600 6650 3600
+	7650 4250 7650 4100
+Wire Wire Line
+	7650 4100 7650 3950
+Wire Wire Line
+	6250 3600 6400 3600
+Wire Wire Line
+	6400 3600 6650 3600
 Wire Wire Line
 	6100 4100 5850 4100
@@
 Connection ~ 6400 5000
 Wire Wire Line
-	5850 3600 5850 4500
-Wire Wire Line
-	5850 4500 3850 4500
+	5850 3600 5850 4100
+Wire Wire Line
+	5850 4100 5850 4500
+Wire Wire Line
+	5850 4500 4200 4500
+Wire Wire Line
+	4200 4500 3850 4500
 Connection ~ 4200 4500
 Connection ~ 5850 4100
@@
 Connection ~ 8700 5000
 Wire Wire Line
-	5950 3100 2600 3100
+	5950 3100 5400 3100
+Wire Wire Line
+	5400 3100 5200 3100
+Wire Wire Line
+	5200 3100 2850 3100
+Wire Wire Line
+	2850 3100 2600 3100
 Wire Wire Line
 	3350 4750 3350 5000
-Text GLabel 2600 3100 0    60   Input ~ 0
-+12V
 $Comp
 L INDUCTOR L2
@@
 +170V
 $Comp
-L GND #PWR2
-U 1 1 52ECE132
-P 9200 5000
-F 0 "#PWR2" H 9200 5000 30  0001 C CNN
-F 1 "GND" H 9200 4930 30  0001 C CNN
-	1    9200 5000
-	0    -1   -1   0
-$EndComp
-$Comp
 L R R5
 U 1 1 52ECE108
@@
 	1    0    0    -1
 $EndComp
-$Comp
-L GND #PWR1
-U 1 1 52ECDB44
-P 2450 5000
-F 0 "#PWR1" H 2450 5000 30  0001 C CNN
-F 1 "GND" H 2450 4930 30  0001 C CNN
-	1    2450 5000
-	0    1    1    0
-$EndComp
 $EndSCHEMATC

Commit message: power_supply: created the net file
Changed lines of the file:
@@
-EESchema Schematic File Version 2  date 2014年02月01日 (週六) 21時51分08秒
+EESchema Schematic File Version 2  date 2014年02月01日 (週六) 21時56分09秒
 LIBS:power
 LIBS:device
@@
 $EndDescr
 $Comp
-L GNDPWR #PWR?
+L GNDPWR #PWR01
 U 1 1 52ECFBB9
 P 2600 5000
-F 0 "#PWR?" H 2600 5050 40  0001 C CNN
+F 0 "#PWR01" H 2600 5050 40  0001 C CNN
 F 1 "GNDPWR" H 2600 4920 40  0000 C CNN
 	1    2600 5000
@@
 $EndComp
 $Comp
-L +12V #PWR?
+L +12V #PWR02
 U 1 1 52ECFBAD
 P 2600 3100
-F 0 "#PWR?" H 2600 3050 20  0001 C CNN
+F 0 "#PWR02" H 2600 3050 20  0001 C CNN
 F 1 "+12V" H 2600 3200 30  0000 C CNN
 	1    2600 3100
@@
 $EndComp
 Wire Wire Line
-	8700 5000 8100 5000
-Wire Wire Line
-	8100 5000 7650 5000
-Wire Wire Line
-	7650 5000 6950 5000
-Wire Wire Line
-	6950 5000 6400 5000
-Wire Wire Line
-	6400 5000 4200 5000
-Wire Wire Line
-	4200 5000 3800 5000
-Wire Wire Line
-	3800 5000 3350 5000
-Wire Wire Line
-	3350 5000 2850 5000
-Wire Wire Line
-	2850 5000 2600 5000
+	2600 5000 8700 5000
 Wire Wire Line
 	3350 4350 3350 4000
@@
 	2850 2900 5600 2900
 Wire Wire Line
-	2850 2900 2850 3100
-Wire Wire Line
-	2850 3100 2850 4000
+	2850 4000 2850 2900
 Connection ~ 2850 5000
 Wire Wire Line
@@
 	6950 5000 6950 3800
 Wire Wire Line
-	3850 3850 3850 4500
+	3850 4500 3850 3850
 Wire Wire Line
 	3850 3850 4050 3850
@@
 	7650 3450 7650 3100
 Wire Wire Line
-	8100 3850 8100 3100
+	8100 3100 8100 3850
 Wire Wire Line
-	7100 3100 6950 3100
+	7100 3100 6550 3100
 Wire Wire Line
-	6950 3100 6550 3100
-Wire Wire Line
-	8100 3100 7650 3100
-Wire Wire Line
-	7650 3100 7500 3100
+	7500 3100 8100 3100
 Wire Wire Line
 	8700 3100 8700 3850
 Wire Wire Line
-	7650 4250 7650 4100
+	7650 4250 7650 3950
 Wire Wire Line
-	7650 4100 7650 3950
-Wire Wire Line
-	6250 3600 6400 3600
-Wire Wire Line
-	6400 3600 6650 3600
+	6250 3600 6650 3600
 Wire Wire Line
 	6100 4100 5850 4100
@@
 Connection ~ 6400 5000
 Wire Wire Line
-	5850 3600 5850 4100
+	5850 4500 5850 3600
 Wire Wire Line
-	5850 4100 5850 4500
-Wire Wire Line
-	5850 4500 4200 4500
-Wire Wire Line
-	4200 4500 3850 4500
+	3850 4500 5850 4500
 Connection ~ 4200 4500
 Connection ~ 5850 4100
@@
 Connection ~ 8700 5000
 Wire Wire Line
-	5950 3100 5400 3100
-Wire Wire Line
-	5400 3100 5200 3100
-Wire Wire Line
-	5200 3100 2850 3100
-Wire Wire Line
-	2850 3100 2600 3100
+	5950 3100 2600 3100
 Wire Wire Line
 	3350 4750 3350 5000
