File: circuit/all_in_one/nixie_control.sch (KiCad schematic (older format))
At the start: 29 parts, among them IC1 ATMEGA328P-A, P1 CONN_01X08, P2 CONN_02X03, P3 CONN_01X12, P4 CONN_02X04, Q3 Q_NPN_EBC, Q4 Q_NPN_EBC, SW1 SW_PUSH, U18 DFPlayer, U3 TLP521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

Commit message: Redesign the all in one board
Parts:
- removed P2: CONN_02X03, Pin_Headers:Pin_Header_Straight_2x03, symbol CONN_02X03
- removed P4: CONN_02X04, Pin_Headers:Pin_Header_Straight_2x04, symbol CONN_02X04
- removed R13, R14: 330ohm, Resistors_SMD:R_0805_HandSoldering, symbol R
- added C13: 0.1uf, Capacitors_SMD:C_0805_HandSoldering, symbol C
- added P2: CONN_01X02, Pin_Headers:Pin_Header_Straight_1x02, symbol CONN_01X02
- added P4: CONN_01X05, Socket_Strips:Socket_Strip_Angled_1x05, symbol CONN_01X05
- added P7: CONN_01X04, Pin_Headers:Pin_Header_Straight_1x04, symbol CONN_01X04
- R10, R11, R12, R15, R18, R19, R8, R9: footprint Resistors_SMD:R_0805_HandSoldering -> Resistors_SMD:R_1206_HandSoldering
- U3, U4, U6, U7: footprint SMD_Packages:DIP-8_SMD -> Housings_DIP:DIP-8_W7.62mm
- U5: footprint SMD_Packages:SO-16-N -> Housings_DIP:DIP-16_W7.62mm
Connections:
- net 5V: now also P2.1 (P1), P4.2 (P2), P7.1 (P1)
- net GND: now also P4.3 (P3), P7.2 (P2)
- net Mode_button: now also P2.2 (P2)
- net Reset: now also C13.2
- net USART_RX: now also P4.4 (P4)
- net USART_TX: now also P4.5 (P5)
- net Adjust_button renamed BLUETOOTH_RX
- net BLUETOOTH_RX: now also P7.3 (P3)
- net Search_button renamed BLUETOOTH_TX
- net BLUETOOTH_TX: now also P7.4 (P4)
- new net: C13.1, P4.1 (P1)
Other:
- moved on the sheet: C8, C9, R12, R15, R18, R19, SP1, SW1, U18, Y1
