File: circuit/all_in_one/nixie_control_board.kicad_pcb (KiCad board)
At the start: 2 copper layers, 136.5 x 42.3 mm, 68 parts, among them CON1 BARREL_JACK, IC1 ATMEGA328P-A, P1 CONN_01X08, P2 CONN_02X03, P3 CONN_01X12, P4 CONN_02X04, P5 CONN_01X08, P6 CONN_01X12, Q1 2SB647, Q2 2SK2611, Q3 Q_NPN_EBC, Q4 Q_NPN_EBC, SW1 SW_PUSH, U1 SMD_7805, U10 IN-14, U11 IN-14, U12 IN-14, U13 IN-14, U14 IN-14, U15 IN-14, U16 IN-14, U17 IN-14, U18 DFPlayer, U2 MC34063A, U3 TLP521, U4 TLP521, U5 HEF4028, U6 TLP521, U7 TLP521, U8 K155ID1, U9 DS1307, Y1 16MHZ, Y2 32.768khz

Commit message: Redesign the all in one board
Parts:
- removed R13, R14: 330ohm, Resistors_SMD:R_0805_HandSoldering
- added C11: 1000pf, Capacitors_SMD:C_0805_HandSoldering, F.Cu at (51.7, 131.7)
- added C12: 1000pf, Capacitors_SMD:C_0805_HandSoldering, F.Cu at (51.7, 134.2)
- added C13: 0.1uf, Capacitors_SMD:C_0805_HandSoldering, F.Cu at (169.4, 126.5)
- added P7: CONN_01X04, Pin_Headers:Pin_Header_Straight_1x04, F.Cu at (230.5, 78.2)
- BT1: footprint cr1220_smd:cr1220smd -> Connect:CR2032H
- C1: value 100uf -> 100uf/16v
- C4: value 1500pf -> 1000pf
- P1, P3, U18: moved to F.Cu
- P2: value CONN_02X03 -> CONN_01X02; footprint Pin_Headers:Pin_Header_Straight_2x03 -> Pin_Headers:Pin_Header_Straight_1x02; moved to F.Cu
- P4: value CONN_02X04 -> CONN_01X05; footprint Pin_Headers:Pin_Header_Straight_2x04 -> Socket_Strips:Socket_Strip_Angled_1x05
- R1, R10, R11, R12, R15, R16, R17, R18, R19, R2, R3, R4, R5, R6, R7, R8, R9: footprint Resistors_SMD:R_0805_HandSoldering -> Resistors_SMD:R_1206_HandSoldering
- U3, U4, U6, U7: footprint SMD_Packages:DIP-8_SMD -> Housings_DIP:DIP-8_W7.62mm
- U5: footprint SMD_Packages:SO-16-N -> Housings_DIP:DIP-16_W7.62mm
- U9: footprint Power_Integrations:SO-8 -> Housings_DIP:DIP-8_W7.62mm
- moved U17 224.5 mm to (50.0, -59.5)
- moved U15 158.8 mm to (86.8, -54.4)
- moved P3 157.8 mm to (259.8, 142.2)
- moved U14 143.6 mm to (239.2, -50.6)
- moved U10 137.9 mm to (124.9, -54.4)
- moved U13 136.7 mm to (199.8, -51.9)
- moved U12 133.9 mm to (171.9, -53.1)
- moved U11 131.7 mm to (147.8, -51.9)
- moved U16 127.1 mm to (267.1, -48.0)
- moved P5 121.0 mm to (168.4, -22.9)
- moved U8 120.8 mm to (238.0, 133.7), turned to 90 degrees
- moved IC1 88.3 mm to (230.2, 101.1), turned to 0 degrees
- moved R15 71.9 mm to (191.4, 107.1), turned to 180 degrees
- moved R12 70.3 mm to (167.6, 76.3), turned to 180 degrees
- moved P6 67.9 mm to (120.3, -21.8), turned to 90 degrees
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Connections:
- IC1 pad 1: Search_button -> BLUETOOTH_TX
- IC1 pad 13: (no net) -> Net-(IC1-Pad13)
- IC1 pad 19: (no net) -> Net-(IC1-Pad19)
- IC1 pad 2: Adjust_button -> BLUETOOTH_RX
- IC1 pad 22: (no net) -> Net-(IC1-Pad22)
- P4 pad 1: USART_TX -> Net-(C13-Pad1)
- P4 pad 2: USART_TX -> /RTC/5V
- P4 pad 3: USART_RX -> /RTC/GND
- P4 pad 5: /RTC/GND -> USART_TX
- U18 pad 10: (no net) -> Net-(U18-Pad10)
- U18 pad 11: (no net) -> Net-(U18-Pad11)
- U18 pad 12: (no net) -> Net-(U18-Pad12)
- U18 pad 13: (no net) -> Net-(U18-Pad13)
- U18 pad 14: (no net) -> Net-(U18-Pad14)
- U18 pad 15: (no net) -> Net-(U18-Pad15)
- U18 pad 16: (no net) -> Net-(U18-Pad16)
- U18 pad 4: (no net) -> Net-(U18-Pad4)
- U18 pad 5: (no net) -> Net-(U18-Pad5)
- U18 pad 9: (no net) -> Net-(U18-Pad9)
- U5 pad 5: (no net) -> Net-(U5-Pad5)
- U5 pad 9: (no net) -> Net-(U5-Pad9)
- U9 pad 7: (no net) -> Net-(U9-Pad7)
Routing:
- net /RTC/GND: track 454.6 -> 0.00 mm, vias 9 -> 0
- net /RTC/5V: track 188.7 -> 0.00 mm, vias 4 -> 0
- net Net-(R9-Pad1): track 124.6 -> 0.00 mm, vias 2 -> 0
- net /power_supply/12V: track 82.0 -> 0.00 mm
- net Net-(P1-Pad3): track 68.9 -> 0.00 mm, vias 2 -> 0
- net Net-(P1-Pad4): track 67.7 -> 0.00 mm, vias 2 -> 0
- net Net-(R8-Pad2): track 62.9 -> 0.00 mm
- net /RTC/I2C_SCL: track 57.9 -> 0.00 mm, vias 4 -> 0
- net Font_C: track 54.4 -> 0.00 mm, vias 1 -> 0
- net Net-(P1-Pad5): track 52.0 -> 0.00 mm
- net /RTC/I2C_SDA: track 51.0 -> 0.00 mm, vias 2 -> 0
- net Net-(P1-Pad2): track 50.5 -> 0.00 mm, vias 2 -> 0
- net Net-(P1-Pad1): track 50.1 -> 0.00 mm, vias 2 -> 0
- net Net-(P1-Pad6): track 49.0 -> 0.00 mm
- net Reset: track 47.8 -> 0.00 mm, vias 2 -> 0
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Other:
- board outline removed
