File: circuit/all_in_one/RTC.sch (KiCad schematic (older format))
At the start: 6 parts, among them U9 DS1307, Y2 32.768khz

Commit message: New hardware is almost finished
Parts:
- BT1: footprint cr1220_smd:cr1220smd -> Connect:CR2032H
- R16, R17: footprint Resistors_SMD:R_0805_HandSoldering -> Resistors_SMD:R_1206_HandSoldering
- U9: footprint Power_Integrations:SO-8 -> Housings_DIP:DIP-8_W7.62mm
Changed lines of the file:
@@
 $Descr A4 11693 8268
 encoding utf-8
-Sheet 4 5
+Sheet 4 4
 Title ""
 Date ""
@@
 F 0 "U9" H 5600 4550 60  0000 C CNN
 F 1 "DS1307" H 5900 4550 60  0000 C CNN
-F 2 "Power_Integrations:SO-8" H 5600 4550 60  0001 C CNN
+F 2 "Housings_DIP:DIP-8_W7.62mm" H 5600 4550 60  0001 C CNN
 F 3 "" H 5600 4550 60  0000 C CNN
 	1    5800 4150
@@
 F 0 "BT1" H 4600 4250 50  0000 L CNN
 F 1 "CR1220" H 4600 4150 50  0000 L CNN
-F 2 "cr1220_smd:cr1220smd" V 4500 4240 60  0001 C CNN
+F 2 "Connect:CR2032H" V 4500 4240 60  0001 C CNN
 F 3 "" V 4500 4240 60  0000 C CNN
 	1    4500 4200
@@
 F 0 "R17" V 7130 4150 50  0000 C CNN
 F 1 "4.7k ohm" V 7050 4150 50  0000 C CNN
-F 2 "Resistors_SMD:R_0805_HandSoldering" V 6980 4150 30  0001 C CNN
+F 2 "Resistors_SMD:R_1206_HandSoldering" V 6980 4150 30  0001 C CNN
 F 3 "" H 7050 4150 30  0000 C CNN
 	1    7050 4150
@@
 F 0 "R16" V 6530 4050 50  0000 C CNN
 F 1 "4.7k ohm" V 6450 4050 50  0000 C CNN
-F 2 "Resistors_SMD:R_0805_HandSoldering" V 6380 4050 30  0001 C CNN
+F 2 "Resistors_SMD:R_1206_HandSoldering" V 6380 4050 30  0001 C CNN
 F 3 "" H 6450 4050 30  0000 C CNN
 	1    6450 4050
