File: circuit/new_design/control_board/RTC.sch (KiCad schematic (older format))
At the start: 6 parts, among them U9 DS1307, Y2 32.768khz

Commit message: Elimanate control board to 2 layers only
Parts:
- BT1: footprint Connect:CR2032H -> CR2032H:CR2032H
Changed lines of the file:
@@
 F 0 "BT1" H 4600 4250 50  0000 L CNN
 F 1 "CR1220" H 4600 4150 50  0000 L CNN
-F 2 "Connect:CR2032H" V 4500 4240 60  0001 C CNN
+F 2 "CR2032H:CR2032H" V 4500 4240 60  0001 C CNN
 F 3 "" V 4500 4240 60  0000 C CNN
 	1    4500 4200
