File: circuit/new_design/control_board/nixie_control_board.kicad_pcb (KiCad board)
At the start: 4 copper layers, 177.9 x 57.6 mm, 62 parts, among them CON1 BARREL_JACK, IC1 ATMEGA328P-A, P1 CONN_01X08, P2 CONN_02X03, P3 CONN_01X12, P4 CONN_01X04, P5 BLUETOOTH_SJ, Q1 2SB647, Q2 2SK2611, Q3 Q_NPN_EBC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

Commit message: Control board is almost finished
Parts:
- added REF**: Symbol_HighVoltage_Type2_CopperTop_VerySmall, warning:warning, F.Cu at (69.3, 124.2)
- added REF**: Pin_Header_Straight_2x04, Pin_Headers:Pin_Header_Straight_2x04, F.Cu at (143.4, 85.6)
- added REF**: Pin_Header_Straight_2x06, Pin_Headers:Pin_Header_Straight_2x06, F.Cu at (158.7, 85.6)
- added REF**: Pin_Header_Straight_2x03, Pin_Headers:Pin_Header_Straight_2x03, F.Cu at (179.0, 85.6)
- BT1: footprint Connect:CR2032H -> CR2032H:CR2032H
- moved U18 2.00 mm to (201.9, 125.2)
- moved P1 0.25 mm to (143.4, 85.6)
- moved P2 0.25 mm to (179.0, 85.6)
- moved P3 0.25 mm to (158.7, 85.6)
Routing:
- net _cathode_comma_left: track 0.00 -> 71.8 mm, vias 0 -> 1
- net /RTC/5V: track 265.3 -> 328.3 mm
- net Net-(BT1-Pad1): track 0.00 -> 18.3 mm
- net Net-(P3-Pad6): track 50.7 -> 46.0 mm
- net Net-(SP1-Pad1): track 33.6 -> 37.6 mm
- net /RTC/GND: track 570.2 -> 573.7 mm
- net Net-(SP1-Pad2): track 41.2 -> 43.7 mm
- net Net-(R18-Pad1): track 35.6 -> 37.8 mm
- net Net-(R19-Pad1): track 27.7 -> 29.4 mm
Other:
- board size 177.9 x 57.6 mm -> 177.9 x 59.4 mm

Commit message: Finish new version hardware design
Parts:
- added REF**: Symbol_HighVoltage_Type2_CopperTop_VerySmall, warning:warning, B.Cu at (68.3, 122.6)
- added REF**: MountingHole_2.2mm_M2, Mounting_Holes:MountingHole_2.2mm_M2, F.Cu at (231.8, 129.8)
- added REF**: MountingHole_2.2mm_M2, Mounting_Holes:MountingHole_2.2mm_M2, F.Cu at (231.8, 80.0)
- added REF**: MountingHole_2.2mm_M2, Mounting_Holes:MountingHole_2.2mm_M2, F.Cu at (56.1, 129.6)
- added REF**: MountingHole_2.2mm_M2, Mounting_Holes:MountingHole_2.2mm_M2, F.Cu at (56.1, 80.0)
- moved D2 20.7 mm to (119.6, 82.0)
- moved BT1 1.02 mm to (158.7, 119.6)
- moved P1 1.02 mm to (142.4, 85.6)
- moved P2 1.02 mm to (178.0, 85.6)
- moved Q3 1.02 mm to (132.9, 82.1)
- moved R12 1.02 mm to (193.9, 84.0)
- moved REF** 1.02 mm to (142.4, 85.6)
- moved REF** 1.02 mm to (178.0, 85.6)
- moved U9 1.02 mm to (186.6, 128.7)
- moved C11 1.02 mm to (78.0, 111.3)
- moved C12 1.02 mm to (74.3, 110.1)
- moved C4 1.02 mm to (78.0, 108.8)
- moved C5 1.02 mm to (77.7, 99.3)
- moved L1 1.02 mm to (94.2, 100.5)
- moved Q1 1.02 mm to (95.4, 106.9)
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- renumbered P5 to BLUETOOTH, U18 to DFPlayer
Routing:
- net /RTC/5V: track 328.3 -> 290.8 mm
- net Net-(SP1-Pad1): track 37.6 -> 66.8 mm
- net /RTC/GND: track 573.7 -> 546.8 mm
- net Net-(D2-Pad2): track 14.5 -> 35.3 mm
- net Net-(SP1-Pad2): track 43.7 -> 63.2 mm
- net Net-(D1-Pad1): track 19.9 -> 33.3 mm
- net USART_TX: track 59.4 -> 54.0 mm
- net USART_RX: track 71.9 -> 66.4 mm
- net Net-(R18-Pad1): track 37.8 -> 33.6 mm
- net Net-(R19-Pad1): track 29.4 -> 33.1 mm
- net /power_supply/12V: track 62.8 -> 60.0 mm, vias 1 -> 0
- added copper zone on B.Cu, net (none)
- added copper zone on F.Cu, net (none)
- added copper zone on In1.Cu, net (none)
- added copper zone on In2.Cu, net (none)
Other:
- board size 177.9 x 59.4 mm -> 183.8 x 59.4 mm
- rule trace_min: 0.2 -> 0.25

Commit message: Elimanate control board to 2 layers only
Parts:
- renumbered BLUETOOTH to P5, DFPlayer to U18
Routing:
- net Net-(P1-Pad6): track 55.6 -> 92.4 mm, vias 1 -> 2
- net Net-(P1-Pad1): track 53.4 -> 87.8 mm, vias 1 -> 2
- net Net-(P1-Pad5): track 39.1 -> 71.1 mm, vias 1 -> 2
- net Net-(U3-Pad1): track 51.9 -> 79.2 mm, vias 0 -> 2
- net Net-(P3-Pad10): track 80.6 -> 57.5 mm
- net Net-(P3-Pad8): track 69.9 -> 56.3 mm
- net Net-(SP1-Pad1): track 66.8 -> 79.6 mm
- net Net-(P3-Pad1): track 54.4 -> 44.3 mm
- net _cathode_comma_left: track 71.8 -> 62.2 mm
- net Net-(P3-Pad2): track 57.4 -> 49.1 mm, vias 1 -> 2
- net /RTC/5V: track 290.8 -> 283.8 mm, vias 5 -> 7
- net Net-(P1-Pad3): track 69.5 -> 75.9 mm, vias 1 -> 2
- net Net-(P3-Pad7): track 29.6 -> 34.4 mm
- net Net-(P3-Pad9): track 47.1 -> 51.8 mm
- net Net-(R9-Pad1): track 80.1 -> 84.8 mm, vias 0 -> 1
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- removed copper zone on In1.Cu, net (none)
- removed copper zone on In2.Cu, net (none)
Other:
- copper layers 4 -> 2
