File: circuit/commertial_design/tube/nixie_control_board.kicad_pcb (KiCad board)
At the start: 2 copper layers, 19.4 x 19.4 mm, 4 parts, among them P1 CONN_01X04, P2 CONN_01X04, P3 CONN_01X05, U10 IN-14

Commit message: Fix PCB board
Changed lines of the file:
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@@
     (links 13)
     (no_connects 0)
-    (area -13.333333 -12.405 13.333334 13.333333)
+    (area -13.333333 -9.875001 13.333334 13.333333)
     (thickness 1.6)
     (drawings 4)
@@
     (visible_elements FFFFFF7F)
     (pcbplotparams
-      (layerselection 0x01030_80000001)
+      (layerselection 0x010f0_80000001)
       (usegerberextensions true)
       (excludeedgelayer true)
@@
       (drillshape 0)
       (scaleselection 1)
-      (outputdirectory 2016_9_13_TUBE/))
+      (outputdirectory TUBE_VER3/))
   )
   (net 0 "")
@@
     (descr "Through hole pin header")
     (tags "pin header")
-    (fp_text reference P1 (at 0 5.1 180) (layer B.SilkS)
-      (effects (font (size 1 1) (thickness 0.15)) (justify mirror))
+    (fp_text reference P1 (at 0.49712 2.65684 180) (layer F.SilkS)
+      (effects (font (size 1 1) (thickness 0.15)))
     )
     (fp_text value CONN_01X04 (at 0 3.1 180) (layer B.Fab) hide
@@
     (descr "Through hole pin header")
     (tags "pin header")
-    (fp_text reference P2 (at 0 5.1 180) (layer B.SilkS)
-      (effects (font (size 1 1) (thickness 0.15)) (justify mirror))
+    (fp_text reference P2 (at -0.86288 2.65684 180) (layer F.SilkS)
+      (effects (font (size 1 1) (thickness 0.15)))
     )
     (fp_text value CONN_01X04 (at 0 3.1 180) (layer B.Fab) hide
@@
     (descr "Through hole pin header")
     (tags "pin header")
-    (fp_text reference P3 (at 0 5.1 270) (layer B.SilkS)
-      (effects (font (size 1 1) (thickness 0.15)) (justify mirror))
+    (fp_text reference P3 (at -0.46156 -12.88288 360) (layer F.SilkS)
+      (effects (font (size 1 1) (thickness 0.15)))
     )
     (fp_text value CONN_01X05 (at 0 3.1 270) (layer B.Fab) hide
@@
   (module IN-14:IN-14 (layer F.Cu)
     (at 0 0)
-    (fp_text reference U10 (at 0.5 -11.43) (layer F.SilkS)
-      (effects (font (size 1 1) (thickness 0.15)))
-    )
+    (fp_text reference U10 (at 0.18288 -1.05156) (layer F.SilkS)
+      (effects (font (size 1 1) (thickness 0.15)))
+    )
