File: circuit/commertial_design/control_board/RTC.sch (KiCad schematic (older format))
At the start: 5 parts, among them U9 DS3231

Commit message: Layout need to be arranged, scheme is finished
Parts:
- BT1: value CR1220 -> CR2032
Changed lines of the file:
@@
 P 7100 3950
 F 0 "BT1" H 7200 4000 50  0000 L CNN
-F 1 "CR1220" H 7200 3900 50  0000 L CNN
+F 1 "CR2032" H 7200 3900 50  0000 L CNN
 F 2 "CR2032H:CR2032H" V 7100 3990 60  0001 C CNN
 F 3 "" V 7100 3990 60  0000 C CNN

Commit message: Fix PCB board
Parts:
- BT1: symbol Battery -> Battery-RESCUE-nixie_control_board
- U9: footprint SMD_Packages:SO-16-N -> SMD_Packages:SO-16-W
Changed lines of the file:
@@
 F 0 "U9" H 6150 3350 60  0000 C CNN
 F 1 "DS3231" H 5850 3350 60  0000 C CNN
-F 2 "SMD_Packages:SO-16-N" H 6100 3350 60  0001 C CNN
+F 2 "SMD_Packages:SO-16-W" H 6100 3350 60  0001 C CNN
 F 3 "" H 6100 3350 60  0000 C CNN
 	1    5900 3250
@@
 	6850 3500 6450 3500
 $Comp
-L Battery BT1
+L Battery-RESCUE-nixie_control_board BT1
 U 1 1 579B979A
 P 7100 3950
