File: circuit/commertial_design/control_board/nixie_control_board.kicad_pcb (KiCad board)
At the start: 2 copper layers, 200 x 66 mm, 77 parts, among them CON1 BARREL_JACK, IC1 ATMEGA328P-A, P1 CONN_01X08, P2 CONN_02X01, P3 CONN_01X12, P4 CONN_01X04, P5 BLUETOOTH_SJ, P6 CONN_02X03, Q1 2SB647, Q2 2SK3611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

Commit message: Fix board errors
Parts:
- removed P5: BLUETOOTH_SJ, HC06:HC06
- removed SW2: SPST, SMD_SOLD_BRIDGE:SMD_BRIDGE
- added C11: 10uf, Capacitors_SMD:C_0805_HandSoldering, F.Cu at (204.5, 76.2)
- added C16: 10uf, Capacitors_SMD:C_0805_HandSoldering, F.Cu at (204.5, 73.7)
- added U10: LM1117-3.3, TO_SOT_Packages_SMD:SOT-223, F.Cu at (211.5, 76.2)
- added U11: hc06, hc06:hc06, F.Cu at (231.8, 79.4)
- moved CON1 0.27 mm to (56.1, 102.1)
Routing:
- net /nixie_control/3V3: track 0.00 -> 69.5 mm
- net /RTC/GND: track 811.5 -> 840.7 mm, vias 7 -> 8
- net USART_RX: track 77.2 -> 104.9 mm, vias 1 -> 2
- net /RTC/5V: track 380.3 -> 394.7 mm, vias 5 -> 7
- net Net-(P5-Pad4): track 5.46 -> 0.00 mm
- net USART_TX: track 72.6 -> 75.8 mm, vias 1 -> 2
- net /power_supply/12V: track 88.0 -> 89.5 mm
